Commit message: v0.3

File: kuka_iiwa_14_support/urdf/kuka_iiwa_14.xacro (robot description, xacro)
@@ -11,14 +11,7 @@
     <xacro:include filename="$(find kuka_iiwa_14_support)/urdf/kuka_iiwa_14_gazebo.xacro"/>
     <xacro:include filename="$(find kuka_iiwa_14_support)/urdf/kuka_iiwa_14_macro.xacro"/>
-    <xacro:include filename="$(find kuka_iiwa_14_support)/urdf/kuka_iiwa_14_transmission.xacro"
-                   arg="${control_type}"/>
+    <xacro:include filename="$(find kuka_iiwa_14_support)/urdf/kuka_iiwa_14_transmission.xacro"/>
     <xacro:kuka_iiwa_14 prefix=""/>
-    <xacro:kuka_iiwa_14_transmission prefix=""/>
+    <xacro:kuka_iiwa_14_transmission prefix="" control_type="$(arg control_type)"/>
     <xacro:kuka_iiwa_14_gazebo prefix=""/>
-    <link name="world"/>
-    <joint name="world_joint" type="fixed">
-        <parent link="world"/>
-        <child link="base_link"/>
-        <origin xyz="0.0 0.0 0.0" rpy="0.0 0.0 0.0"/>
-    </joint>
 </robot>

File: kuka_iiwa_14_support/urdf/kuka_iiwa_14_macro.xacro (robot description, xacro)
@@ -2,25 +2,12 @@
 <robot xmlns:xacro="http://wiki.ros.org/xacro">
     <xacro:macro name="kuka_iiwa_14" params="prefix">
-        <!-- some constants -->
-        <xacro:property name="max_effort" value="300"/>
-        <xacro:property name="max_velocity" value="10"/>
-        <xacro:property name="damping_factor" value="0.1"/>
-        <xacro:property name="d0" value="${damping_factor*0.1}"/>
-        <xacro:property name="d1" value="${damping_factor*0.1}"/>
-        <xacro:property name="d2" value="${damping_factor*0.1}"/>
-        <xacro:property name="d3" value="${damping_factor*0.1}"/>
-        <xacro:property name="d4" value="${damping_factor*0.1}"/>
-        <xacro:property name="d5" value="${damping_factor*0.1}"/>
-        <xacro:property name="d6" value="${damping_factor*0.1}"/>
-        <xacro:property name="friction_factor" value="0.1"/>
-        <xacro:property name="f0" value="${friction_factor*0.1}"/>
-        <xacro:property name="f1" value="${friction_factor*0.1}"/>
-        <xacro:property name="f2" value="${friction_factor*0.1}"/>
-        <xacro:property name="f3" value="${friction_factor*0.1}"/>
-        <xacro:property name="f4" value="${friction_factor*0.1}"/>
-        <xacro:property name="f5" value="${friction_factor*0.1}"/>
-        <xacro:property name="f6" value="${friction_factor*0.1}"/>
         <xacro:property name="PI" value="3.14"/>
         <!-- ********************* LINKS *********************** -->
+        <link name="world"/>
+        <joint name="world_joint" type="fixed">
+            <parent link="world"/>
+            <child link="base_link"/>
+            <origin xyz="0.0 0.0 0.0" rpy="0.0 0.0 0.0"/>
+        </joint>
         <link name="${prefix}base_link">
             <inertial>
@@ -34,5 +21,4 @@
                     <mesh filename="package://kuka_iiwa_14_support/meshes/visual/link_0.dae"/>
                 </geometry>
-                <material name="Grey"/>
             </visual>
             <collision>
@@ -41,5 +27,4 @@
                     <mesh filename="package://kuka_iiwa_14_support/meshes/collision/link_0.stl"/>
                 </geometry>
-                <material name="Grey"/>
             </collision>
             <self_collision_checking>
@@ -61,5 +46,4 @@
                     <mesh filename="package://kuka_iiwa_14_support/meshes/visual/link_1.dae"/>
                 </geometry>
-                <material name="Orange"/>
             </visual>
             <collision>
@@ -68,5 +52,4 @@
                     <mesh filename="package://kuka_iiwa_14_support/meshes/collision/link_1.stl"/>
                 </geometry>
-                <material name="Orange"/>
             </collision>
         </link>
@@ -82,5 +65,4 @@
                     <mesh filename="package://kuka_iiwa_14_support/meshes/visual/link_2.dae"/>
                 </geometry>
-                <material name="Orange"/>
             </visual>
             <collision>
@@ -89,5 +71,4 @@
                     <mesh filename="package://kuka_iiwa_14_support/meshes/collision/link_2.stl"/>
                 </geometry>
-                <material name="Orange"/>
             </collision>
         </link>
@@ -103,5 +84,4 @@
                     <mesh filename="package://kuka_iiwa_14_support/meshes/visual/link_3.dae"/>
                 </geometry>
-                <material name="Orange"/>
             </visual>
             <collision>
@@ -110,5 +90,4 @@
                     <mesh filename="package://kuka_iiwa_14_support/meshes/collision/link_3.stl"/>
                 </geometry>
-                <material name="Orange"/>
             </collision>
         </link>
@@ -124,5 +103,4 @@
                     <mesh filename="package://kuka_iiwa_14_support/meshes/visual/link_4.dae"/>
                 </geometry>
-                <material name="Orange"/>
             </visual>
             <collision>
@@ -131,5 +109,4 @@
                     <mesh filename="package://kuka_iiwa_14_support/meshes/collision/link_4.stl"/>
                 </geometry>
-                <material name="Orange"/>
             </collision>
         </link>
@@ -145,5 +122,4 @@
                     <mesh filename="package://kuka_iiwa_14_support/meshes/visual/link_5.dae"/>
                 </geometry>
-                <material name="Orange"/>
             </visual>
             <collision>
@@ -152,5 +128,4 @@
                     <mesh filename="package://kuka_iiwa_14_support/meshes/collision/link_5.stl"/>
                 </geometry>
-                <material name="Orange"/>
             </collision>
         </link>
@@ -166,5 +141,4 @@
                     <mesh filename="package://kuka_iiwa_14_support/meshes/visual/link_6.dae"/>
                 </geometry>
-                <material name="Orange"/>
             </visual>
             <collision>
@@ -173,5 +147,4 @@
                     <mesh filename="package://kuka_iiwa_14_support/meshes/collision/link_6.stl"/>
                 </geometry>
-                <material name="Orange"/>
             </collision>
         </link>
@@ -187,5 +160,4 @@
                     <mesh filename="package://kuka_iiwa_14_support/meshes/visual/link_7.dae"/>
                 </geometry>
-                <material name="Grey"/>
             </visual>
             <collision>
@@ -194,5 +166,4 @@
                     <mesh filename="package://kuka_iiwa_14_support/meshes/collision/link_7.stl"/>
                 </geometry>
-                <material name="Grey"/>
             </collision>
         </link>
@@ -206,6 +177,6 @@
             <axis xyz="0 0 1"/>
             <limit lower="${-170 * PI / 180}" upper="${170 * PI / 180}"
-                   effort="${max_effort}" velocity="${max_velocity}"/>
-            <dynamics damping="${d0}" friction="${f0}"/>
+                   effort="300" velocity="10"/>
+            <dynamics damping="0.1" friction="0.1"/>
         </joint>
         <joint name="${prefix}joint_2" type="revolute">
@@ -215,6 +186,6 @@
             <axis xyz="0 0 1"/>
             <limit lower="${-120 * PI / 180}" upper="${120 * PI / 180}"
-                   effort="${max_effort}" velocity="${max_velocity}"/>
-            <dynamics damping="${d1}" friction="${f1}"/>
+                          effort="300" velocity="10"/>
+            <dynamics damping="0.1" friction="0.1"/>
         </joint>
         <joint name="${prefix}joint_3" type="revolute">
@@ -224,6 +195,6 @@
             <axis xyz="0 0 1"/>
             <limit lower="${-170 * PI / 180}" upper="${170 * PI / 180}"
-                   effort="${max_effort}" velocity="${max_velocity}"/>
-            <dynamics damping="${d2}" friction="${f2}"/>
+                           effort="300" velocity="10"/>
+            <dynamics damping="0.1" friction="0.1"/>
         </joint>
         <joint name="${prefix}joint_4" type="revolute">
@@ -233,6 +204,6 @@
             <axis xyz="0 0 1"/>
             <limit lower="${-120 * PI / 180}" upper="${120 * PI / 180}"
-                   effort="${max_effort}" velocity="${max_velocity}"/>
-            <dynamics damping="${d3}" friction="${f3}"/>
+                          effort="300" velocity="10"/>
+            <dynamics damping="0.1" friction="0.1"/>
         </joint>
         <joint name="${prefix}joint_5" type="revolute">
@@ -242,6 +213,6 @@
             <axis xyz="0 0 1"/>
             <limit lower="${-170 * PI / 180}" upper="${170 * PI / 180}"
-                   effort="${max_effort}" velocity="${max_velocity}"/>
-            <dynamics damping="${d4}" friction="${f4}"/>
+                          effort="300" velocity="10"/>
+            <dynamics damping="0.1" friction="0.1"/>
         </joint>
         <joint name="${prefix}joint_6" type="revolute">
@@ -251,6 +222,6 @@
             <axis xyz="0 0 1"/>
             <limit lower="${-120 * PI / 180}" upper="${120 * PI / 180}"
-                   effort="${max_effort}" velocity="${max_velocity}"/>
-            <dynamics damping="${d5}" friction="${f5}"/>
+                      effort="300" velocity="10"/>
+            <dynamics damping="0.1" friction="0.1"/>
         </joint>
         <joint name="${prefix}joint_7" type="revolute">
@@ -260,6 +231,6 @@
             <axis xyz="0 0 1"/>
             <limit lower="${-175 * PI / 180}" upper="${175 * PI / 180}"
-                   effort="${max_effort}" velocity="${max_velocity}"/>
-            <dynamics damping="${d6}" friction="${f6}"/>
+                           effort="300" velocity="10"/>
+            <dynamics damping="0.1" friction="0.1"/>
         </joint>
         <joint name="${prefix}joint_7-tool0" type="fixed">

File: kuka_iiwa_14_support/urdf/kuka_iiwa_14_transmission.xacro (robot description, xacro)
@@ -1,13 +1,12 @@
 <?xml version="1.0"?>
 <robot xmlns:xacro="http://wiki.ros.org/xacro">
-    <xacro:macro name="kuka_iiwa_14_transmission" params="prefix">
-        <xacro:arg name="control_type" default="Position"/>
+    <xacro:macro name="kuka_iiwa_14_transmission" params="prefix control_type">
         <transmission name="${prefix}effort_tran1">
             <type>transmission_interface/SimpleTransmission</type>
             <joint name="${prefix}joint_1">
-                <hardwareInterface>hardware_interface/$(arg control_type)JointInterface</hardwareInterface>
+                <hardwareInterface>hardware_interface/${control_type}JointInterface</hardwareInterface>
             </joint>
             <actuator name="${prefix}motor1">
-                <hardwareInterface>hardware_interface/$(arg control_type)JointInterface</hardwareInterface>
+                <hardwareInterface>hardware_interface/${control_type}JointInterface</hardwareInterface>
                 <mechanicalReduction>1</mechanicalReduction>
             </actuator>
@@ -16,8 +15,8 @@
             <type>transmission_interface/SimpleTransmission</type>
             <joint name="${prefix}joint_2">
-                <hardwareInterface>hardware_interface/$(arg control_type)JointInterface</hardwareInterface>
+                <hardwareInterface>hardware_interface/${control_type}JointInterface</hardwareInterface>
             </joint>
             <actuator name="${prefix}motor2">
-                <hardwareInterface>hardware_interface/$(arg control_type)JointInterface</hardwareInterface>
+                <hardwareInterface>hardware_interface/${control_type}JointInterface</hardwareInterface>
                 <mechanicalReduction>1</mechanicalReduction>
             </actuator>
@@ -26,8 +25,8 @@
             <type>transmission_interface/SimpleTransmission</type>
             <joint name="${prefix}joint_3">
-                <hardwareInterface>hardware_interface/$(arg control_type)JointInterface</hardwareInterface>
+                <hardwareInterface>hardware_interface/${control_type}JointInterface</hardwareInterface>
             </joint>
             <actuator name="${prefix}motor3">
-                <hardwareInterface>hardware_interface/$(arg control_type)JointInterface</hardwareInterface>
+                <hardwareInterface>hardware_interface/${control_type}JointInterface</hardwareInterface>
                 <mechanicalReduction>1</mechanicalReduction>
             </actuator>
@@ -36,8 +35,8 @@
             <type>transmission_interface/SimpleTransmission</type>
             <joint name="${prefix}joint_4">
-                <hardwareInterface>hardware_interface/$(arg control_type)JointInterface</hardwareInterface>
+                <hardwareInterface>hardware_interface/${control_type}JointInterface</hardwareInterface>
             </joint>
             <actuator name="${prefix}motor4">
-                <hardwareInterface>hardware_interface/$(arg control_type)JointInterface</hardwareInterface>
+                <hardwareInterface>hardware_interface/${control_type}JointInterface</hardwareInterface>
                 <mechanicalReduction>1</mechanicalReduction>
             </actuator>
@@ -46,8 +45,8 @@
             <type>transmission_interface/SimpleTransmission</type>
             <joint name="${prefix}joint_5">
-                <hardwareInterface>hardware_interface/$(arg control_type)JointInterface</hardwareInterface>
+                <hardwareInterface>hardware_interface/${control_type}JointInterface</hardwareInterface>
             </joint>
             <actuator name="${prefix}motor5">
-                <hardwareInterface>hardware_interface/$(arg control_type)JointInterface</hardwareInterface>
+                <hardwareInterface>hardware_interface/${control_type}JointInterface</hardwareInterface>
                 <mechanicalReduction>1</mechanicalReduction>
             </actuator>
@@ -56,8 +55,8 @@
             <type>transmission_interface/SimpleTransmission</type>
             <joint name="${prefix}joint_6">
-                <hardwareInterface>hardware_interface/$(arg control_type)JointInterface</hardwareInterface>
+                <hardwareInterface>hardware_interface/${control_type}JointInterface</hardwareInterface>
             </joint>
             <actuator name="${prefix}motor6">
-                <hardwareInterface>hardware_interface/$(arg control_type)JointInterface</hardwareInterface>
+                <hardwareInterface>hardware_interface/${control_type}JointInterface</hardwareInterface>
                 <mechanicalReduction>1</mechanicalReduction>
             </actuator>
@@ -66,8 +65,8 @@
             <type>transmission_interface/SimpleTransmission</type>
             <joint name="${prefix}joint_7">
-                <hardwareInterface>hardware_interface/$(arg control_type)JointInterface</hardwareInterface>
+                <hardwareInterface>hardware_interface/${control_type}JointInterface</hardwareInterface>
             </joint>
             <actuator name="${prefix}motor7">
-                <hardwareInterface>hardware_interface/$(arg control_type)JointInterface</hardwareInterface>
+                <hardwareInterface>hardware_interface/${control_type}JointInterface</hardwareInterface>
                 <mechanicalReduction>1</mechanicalReduction>
             </actuator>

File: kuka_youbot_support/urdf/kuka_youbot.xacro (robot description, xacro)
@@ -1,11 +1,14 @@
-<?xml version="1.0"?>
+<?xml version="1.0" encoding="UTF-8"?>
 <robot name="kuka_youbot" xmlns:xacro="http://wiki.ros.org/xacro">
     <xacro:arg name="control_type" default="Position"/>
+    <xacro:arg name="main_frame_name" default="footprint"/>
     <!-- Import all Gazebo-customization elements, including Gazebo colors -->
     <xacro:include filename="$(find kuka_youbot_support)/urdf/kuka_youbot_gazebo.xacro"/>
     <xacro:include filename="$(find kuka_youbot_support)/urdf/kuka_youbot_macro.xacro"/>
     <xacro:include filename="$(find kuka_youbot_support)/urdf/kuka_youbot_transmission.xacro"/>
-    <xacro:kuka_youbot prefix=""/>
+    <xacro:kuka_youbot prefix="" main_frame_name="$(arg main_frame_name)"/>
     <xacro:kuka_youbot_transmission prefix="" control_type="$(arg control_type)"/>
-    <xacro:kuka_youbot_gazebo prefix=""/>
+    <xacro:kuka_youbot_gazebo prefix="" main_frame_name="$(arg main_frame_name)"/>
+    <!-- For mobile robots we can not set world as main frame, but rvis requires it. Because of that we need to specify
+    name of main frame with run parameter-->
 </robot>

File: kuka_youbot_support/urdf/kuka_youbot_gazebo.xacro (robot description, xacro)
@@ -1,7 +1,7 @@
-<?xml version="1.0"?>
+<?xml version="1.0"  encoding="UTF-8"?>
 <robot xmlns:xacro="http://wiki.ros.org/xacro">
-    <xacro:macro name="kuka_youbot_gazebo" params="prefix">
+    <xacro:macro name="kuka_youbot_gazebo" params="prefix main_frame_name">
         <!--***********************ARM****************************-->
-         <gazebo>
+        <gazebo>
             <plugin name="gazebo_ros_control" filename="libgazebo_ros_control.so">
                 <robotNamespace>/kuka_youbot</robotNamespace>
@@ -63,5 +63,5 @@
             <material value="youbot/Orange"/>
         </gazebo>
-          <gazebo reference="${prefix}_palm_link">
+        <gazebo reference="${prefix}_palm_link">
             <material>Gazebo/Black</material>
             <turnGravityOff>false</turnGravityOff>
@@ -74,5 +74,5 @@
                 <odometryFrame>/kuka_youbot/odom</odometryFrame>
                 <odometryRate>100.0</odometryRate>
-                <robotBaseFrame>base_footprint</robotBaseFrame>
+                <robotBaseFrame>${prefix}${main_frame_name}</robotBaseFrame>
             </plugin>
         </gazebo>
