Commit message: v0.3

File: kuka_youbot_support/urdf/kuka_youbot_macro.xacro (robot description, xacro)
@@ -1,33 +1,13 @@
-<?xml version="1.0"?>
+<?xml version="1.0"  encoding="UTF-8"?>
 <robot xmlns:xacro="http://wiki.ros.org/xacro">
-    <!-- common properties -->
+    <!-- PI константа -->
     <xacro:property name="PI" value="3.1415926535897931"/>
-    <xacro:property name="threshold" value="0.01"/>
-    <!-- arm limits positions (deg) -->
-    <xacro:property name="joint_1_limit" value="${PI * (169 + 169) / 180}"/>
-    <xacro:property name="joint_2_limit" value="${PI * (90 + 65) / 180}"/>
-    <xacro:property name="joint_3_limit" value="${PI * (146 + 151) / 180}"/>
-    <xacro:property name="joint_4_limit" value="${PI * (102.5 + 102.5) / 180}"/>
-    <xacro:property name="joint_5_limit" value="${PI * (167.5 + 167.5) / 180}"/>
-    <!-- dynamic properties : mass (kg) Alu data sheet -->
-    <xacro:property name="link_0_mass" value="0.845"/>
-    <xacro:property name="link_1_mass" value="2.412"/>
-    <xacro:property name="link_2_mass" value="1.155"/>
-    <xacro:property name="link_3_mass" value="0.934"/>
-    <xacro:property name="link_4_mass" value="0.877"/>
-    <xacro:property name="link_5_mass" value="0.251"/>
-    <!-- simplified box collision geometry for base -->
-    <xacro:property name="base_size_x" value="0.570"/>
-    <xacro:property name="base_size_y" value="0.360"/>
-    <xacro:property name="base_size_z" value="0.100"/>
-    <xacro:property name="base_mass" value="100.0"/>
+    <!--т.к. колёса у нас одинаоквые, а их 4 для экономии места запишем их параметры через переменные-->
     <xacro:property name="caster_offset_x" value="0.228"/>
     <xacro:property name="caster_offset_y" value="0.158"/>
     <xacro:property name="caster_offset_z" value="-0.034"/>
-    <xacro:property name="caster_mass" value="0.1"/>
     <xacro:property name="wheel_offset_x" value="0.0"/>
     <xacro:property name="wheel_offset_y" value="0.0"/>
     <xacro:property name="wheel_offset_z" value="0.0"/>
-    <xacro:property name="wheel_mass" value="0.4"/>
     <xacro:property name="wheel_radius" value="0.05"/>
     <xacro:property name="wheel_length" value="0.005"/>
@@ -36,16 +16,39 @@
     <xacro:property name="caster_joint_effort" value="30"/>
     <xacro:property name="caster_joint_velocity" value="10"/>
-    <xacro:property name="caster_joint_safety_k_velocity" value="10.0"/>
     <xacro:property name="wheel_joint_damping" value="1.0"/>
     <xacro:property name="wheel_joint_friction" value="1.0"/>
     <xacro:property name="wheel_joint_effort" value="30"/>
     <xacro:property name="wheel_joint_velocity" value="10"/>
-    <xacro:property name="wheel_joint_safety_k_velocity" value="10.0"/>
-    <!-- fingers limits, values are in meters -->
-    <xacro:property name="finger_joint" value="${0.023 / 2.0}"/>
-    <xacro:property name="finger_joint_soft" value="${(0.023 - threshold) / 2.0}"/>
-    <xacro:macro name="kuka_youbot" params="prefix">
+    <xacro:macro name="wheel_link_content">
+        <inertial>
+            <mass value="0.4"/>
+            <origin xyz="0 0 0"/>
+            <inertia ixx="0.012411765597" ixy="-0.000711733678" ixz="0.00050272983" iyy="0.015218160428"
+                     iyz="-0.000004273467" izz="0.011763977943"/>
+        </inertial>
+        <visual>
+            <origin xyz="0 0 0" rpy="0 0 0"/>
+            <geometry>
+                <sphere radius="${wheel_radius}"/>
+            </geometry>
+        </visual>
+        <collision>
+            <origin xyz="0 0 0" rpy="${PI/2} 0 0"/>
+            <geometry>
+                <cylinder radius="${wheel_radius}" length="${wheel_radius}"/>
+            </geometry>
+        </collision>
+    </xacro:macro>
+    <xacro:macro name="caster_link_content">
+        <inertial>
+            <mass value="0.1"/>
+            <origin xyz="0 0 0"/>
+            <inertia ixx="0.012411765597" ixy="-0.000711733678" ixz="0.00050272983" iyy="0.015218160428"
+                     iyz="-0.000004273467" izz="0.011763977943"/>
+        </inertial>
+    </xacro:macro>
+    <xacro:macro name="kuka_youbot" params="prefix main_frame_name">
         <!--******************************************BASE*************************************************-->
-        <link name="${prefix}_footprint">
+        <link name="${prefix}${main_frame_name}">
             <visual>
                 <origin xyz="0 0 0" rpy="0 0 0"/>
@@ -55,5 +58,5 @@
             </visual>
             <collision>
-                <origin xyz="0 0 ${-base_size_z / 2.0}" rpy="0 0 0"/>
+                <origin xyz="0 0 -0.050" rpy="0 0 0"/>
                 <geometry>
                     <box size="0.001 0.001 0.001"/>
@@ -76,5 +79,5 @@
                 <origin xyz="0 0 0" rpy="0 0 0"/>
                 <geometry>
-                    <mesh filename="package://kuka_youbot_support/meshes/collision/plate_convex.dae"/>
+                    <mesh filename="package://kuka_youbot_support/meshes/collision/plate.stl"/>
                 </geometry>
             </collision>
@@ -82,5 +85,5 @@
         <link name="${prefix}base_link">
             <inertial>
-                <mass value="${base_mass}"/>
+                <mass value="100"/>
                 <origin xyz="0 0 0"/>
                 <inertia ixx="5.652232699207" ixy="-0.009719934438" ixz="1.293988226423" iyy="5.669473158652"
@@ -96,119 +99,31 @@
                 <origin xyz="0 0 0" rpy="0 0 0"/>
                 <geometry>
-                   <mesh filename="package://kuka_youbot_support/meshes/collision/base_convex.dae"/>
+                    <mesh filename="package://kuka_youbot_support/meshes/collision/base.stl"/>
                 </geometry>
             </collision>
         </link>
         <link name="caster_link_fl">
-            <inertial>
-                <mass value="${caster_mass}"/>
-                <origin xyz="0 0 0"/>
-                <inertia ixx="0.012411765597" ixy="-0.000711733678" ixz="0.00050272983" iyy="0.015218160428"
-                         iyz="-0.000004273467" izz="0.011763977943"/>
-            </inertial>
+            <xacro:caster_link_content/>
         </link>
         <link name="wheel_link_fl">
-            <inertial>
-                <mass value="${wheel_mass}"/>
-                <origin xyz="0 0 0"/>
-                <inertia ixx="0.012411765597" ixy="-0.000711733678" ixz="0.00050272983" iyy="0.015218160428"
-                         iyz="-0.000004273467" izz="0.011763977943"/>
-            </inertial>
-            <visual>
-                <origin xyz="0 0 0" rpy="0 0 0"/>
-                 <geometry>
-                    <sphere radius="${wheel_radius}"/>
-                </geometry>
-            </visual>
-            <collision>
-                <origin xyz="0 0 0" rpy="${PI/2} 0 0"/>
-                <geometry>
-                    <cylinder radius="${wheel_radius}" length="${wheel_radius}"/>
-                </geometry>
-            </collision>
+            <xacro:wheel_link_content/>
         </link>
         <link name="caster_link_fr">
-            <inertial>
-                <mass value="${caster_mass}"/>
-                <origin xyz="0 0 0"/>
-                <inertia ixx="0.012411765597" ixy="-0.000711733678" ixz="0.00050272983" iyy="0.015218160428"
-                         iyz="-0.000004273467" izz="0.011763977943"/>
-            </inertial>
+            <xacro:caster_link_content/>
         </link>
         <link name="wheel_link_fr">
-            <inertial>
-                <mass value="${wheel_mass}"/>
-                <origin xyz="0 0 0"/>
-                <inertia ixx="0.012411765597" ixy="-0.000711733678" ixz="0.00050272983" iyy="0.015218160428"
-                         iyz="-0.000004273467" izz="0.011763977943"/>
-            </inertial>
-            <visual>
-                <origin xyz="0 0 0" rpy="0 0 0"/>
-                <geometry>
-                    <sphere radius="${wheel_radius}"/>
-                </geometry>
-            </visual>
-            <collision>
-                <origin xyz="0 0 0" rpy="${PI/2} 0 0"/>
-                <geometry>
-                    <cylinder radius="${wheel_radius}" length="${wheel_radius}"/>
-                </geometry>
-            </collision>
+            <xacro:wheel_link_content/>
         </link>
         <link name="caster_link_bl">
-            <inertial>
-                <mass value="${caster_mass}"/>
-                <origin xyz="0 0 0"/>
-                <inertia ixx="0.012411765597" ixy="-0.000711733678" ixz="0.00050272983" iyy="0.015218160428"
-                         iyz="-0.000004273467" izz="0.011763977943"/>
-            </inertial>
+            <xacro:caster_link_content/>
         </link>
         <link name="wheel_link_bl">
-            <inertial>
-                <mass value="${wheel_mass}"/>
-                <origin xyz="0 0 0"/>
-                <inertia ixx="0.012411765597" ixy="-0.000711733678" ixz="0.00050272983" iyy="0.015218160428"
-                         iyz="-0.000004273467" izz="0.011763977943"/>
-            </inertial>
-            <visual>
-                <origin xyz="0 0 0" rpy="0 0 0"/>
-                <geometry>
-                     <sphere radius="${wheel_radius}"/>
-                </geometry>
-            </visual>
-            <collision>
-                <origin xyz="0 0 0" rpy="${PI/2} 0 0"/>
-                <geometry>
-                    <cylinder radius="${wheel_radius}" length="${wheel_radius}"/>
-                </geometry>
-            </collision>
+            <xacro:wheel_link_content/>
         </link>
         <link name="caster_link_br">
-            <inertial>
-                <mass value="${caster_mass}"/>
-                <origin xyz="0 0 0"/>
-                <inertia ixx="0.012411765597" ixy="-0.000711733678" ixz="0.00050272983" iyy="0.015218160428"
-                         iyz="-0.000004273467" izz="0.011763977943"/>
-            </inertial>
+            <xacro:caster_link_content/>
         </link>
         <link name="wheel_link_br">
-            <inertial>
-                <mass value="${wheel_mass}"/>
-                <origin xyz="0 0 0"/>
-                <inertia ixx="0.012411765597" ixy="-0.000711733678" ixz="0.00050272983" iyy="0.015218160428"
-                         iyz="-0.000004273467" izz="0.011763977943"/>
-            </inertial>
-            <visual>
-                <origin xyz="0 0 0" rpy="0 0 0"/>
-                <geometry>
-                     <sphere radius="${wheel_radius}"/>
-                </geometry>
-            </visual>
-            <collision>
-                <origin xyz="0 0 0" rpy="${PI/2} 0 0"/>
-                <geometry>
-                    <cylinder radius="${wheel_radius}" length="${wheel_radius}"/>
-                </geometry>
-            </collision>
+            <xacro:wheel_link_content/>
         </link>
         <joint name="${prefix}plate_joint" type="fixed">
@@ -217,8 +132,8 @@
             <child link="${prefix}plate_link"/>
         </joint>
-        <joint name="${prefix}_footprint_joint" type="fixed">
+        <joint name="${prefix}footprint_joint" type="fixed">
             <origin xyz="0 0 0" rpy="0 0 0"/>
             <child link="${prefix}base_link"/>
-            <parent link="${prefix}_footprint"/>
+            <parent link="${prefix}${main_frame_name}"/>
         </joint>
         <joint name="caster_joint_fl" type="continuous">
@@ -291,5 +206,5 @@
             <inertial>
                 <origin xyz="0 0 0" rpy="0 0 0"/>
-                <mass value="${link_0_mass}"/>
+                <mass value="0.845"/>
                 <inertia ixx="0.01" ixy="0" ixz="0" iyy="0.01" iyz="0" izz="0.01"/>
             </inertial>
@@ -297,11 +212,11 @@
                 <origin xyz="0 0 0" rpy="0 0 0"/>
                 <geometry>
-                    <mesh filename="package://kuka_youbot_support/meshes/visual/arm0.dae"/>
-                </geometry>
-            </visual>
-            <collision>
-                <origin xyz="0 0 0" rpy="0 0 0"/>
-                <geometry>
-                    <mesh filename="package://kuka_youbot_support/meshes/collision/arm0_convex.dae"/>
+                    <mesh filename="package://kuka_youbot_support/meshes/visual/link_0.dae"/>
+                </geometry>
+            </visual>
+            <collision>
+                <origin xyz="0 0 0" rpy="0 0 0"/>
+                <geometry>
+                    <mesh filename="package://kuka_youbot_support/meshes/collision/link_0.stl"/>
                 </geometry>
             </collision>
@@ -309,6 +224,6 @@
         <link name="${prefix}arm_link_1">
             <inertial>
-                <mass value="${link_1_mass}"/>
-                <origin xyz="${14.89/1000} ${2.13/1000} ${2.13/1000}" rpy="0 0 0"/>
+                <mass value="2.412"/>
+                <origin xyz="0.01489 0.00213 0.00213" rpy="0 0 0"/>
                 <inertia ixx="0.003863" ixy="-0.000979" ixz="0.000000" iyy="0.006196" iyz="0.000000" izz="0.006369"/>
             </inertial>
@@ -316,18 +231,18 @@
                 <origin xyz="0 0 0" rpy="0 0 0"/>
                 <geometry>
-                    <mesh filename="package://kuka_youbot_support/meshes/visual/arm1.dae"/>
-                </geometry>
-            </visual>
-            <collision>
-                <origin xyz="0 0 0" rpy="0 0 0"/>
-                <geometry>
-                    <mesh filename="package://kuka_youbot_support/meshes/collision/arm1_convex.dae"/>
-                </geometry>
-            </collision>
-        </link>
-  <link name="${prefix}arm_link_2">
-            <inertial>
-                <mass value="${link_2_mass}"/>
-                <origin xyz="${104.53/1000} ${1.7/1000} ${-2.97/1000}"
+                    <mesh filename="package://kuka_youbot_support/meshes/visual/link_1.dae"/>
+                </geometry>
+            </visual>
+            <collision>
+                <origin xyz="0 0 0" rpy="0 0 0"/>
+                <geometry>
+                    <mesh filename="package://kuka_youbot_support/meshes/collision/link_1.stl"/>
+                </geometry>
+            </collision>
+        </link>
+        <link name="${prefix}arm_link_2">
+            <inertial>
+                <mass value="1.155"/>
+                <origin xyz="0.10453 0.0017 -0.00297"
                         rpy="0 0 0"/>
                 <inertia ixx="0.000823" ixy="0.000000" ixz="-0.000000" iyy="0.004447" iyz="0.000000" izz="0.004439"/>
@@ -336,5 +251,5 @@
                 <origin xyz="0 -0.032 0.078" rpy="0 0 0"/>
                 <geometry>
-                    <mesh filename="package://kuka_youbot_support/meshes/visual/arm2.dae"/>
+                    <mesh filename="package://kuka_youbot_support/meshes/visual/link_2.dae"/>
                 </geometry>
             </visual>
@@ -342,12 +257,12 @@
                 <origin xyz="0 -0.032 0.078" rpy="0 0 0"/>
                 <geometry>
-                    <mesh filename="package://kuka_youbot_support/meshes/collision/arm2_convex.dae"/>
-                </geometry>
-            </collision>
-        </link>
-         <link name="${prefix}arm_link_3">
-            <inertial>
-                <mass value="${link_3_mass}"/>
-                <origin xyz="${0.1/1000} ${96.7/1000} ${21.07/1000}"
+                    <mesh filename="package://kuka_youbot_support/meshes/collision/link_2.stl"/>
+                </geometry>
+            </collision>
+        </link>
+        <link name="${prefix}arm_link_3">
+            <inertial>
+                <mass value="0.934"/>
+                <origin xyz="0.0001 0.0967 0.02107"
                         rpy="0 0 0"/>
                 <inertia ixx="0.002459" ixy="0.000000" ixz="0.000000" iyy="0.002571" iyz="-0.000000" izz="0.000535"/>
@@ -356,5 +271,5 @@
                 <origin xyz="0.000 0.028 0.079" rpy="0 0 0"/>
                 <geometry>
-                    <mesh filename="package://kuka_youbot_support/meshes/visual/arm3.dae"/>
+                    <mesh filename="package://kuka_youbot_support/meshes/visual/link_3.dae"/>
                 </geometry>
             </visual>
@@ -362,12 +277,12 @@
                 <origin xyz="0.000 0.028 0.079" rpy="0 0 0"/>
                 <geometry>
-                    <mesh filename="package://kuka_youbot_support/meshes/collision/arm3_convex.dae"/>
-                </geometry>
-            </collision>
-        </link>
-         <link name="${prefix}arm_link_4">
-            <inertial>
-                <mass value="${link_4_mass}"/>
-                <origin xyz="${0.11/1000} ${51.03/1000} ${-23.19/1000}"
+                    <mesh filename="package://kuka_youbot_support/meshes/collision/link_3.stl"/>
+                </geometry>
+            </collision>
+        </link>
+        <link name="${prefix}arm_link_4">
+            <inertial>
+                <mass value="0.877"/>
+                <origin xyz="0.00011 0.05103 -0.02319"
                         rpy="0 0 0"/>
                 <inertia ixx="0.000869" ixy="0.000000" ixz="-0.000000" iyy="0.001173" iyz="-0.000231" izz="0.001091"/>
@@ -376,5 +291,5 @@
                 <origin xyz="0 -0.010 0.029" rpy="0 0 0"/>
                 <geometry>
-                    <mesh filename="package://kuka_youbot_support/meshes/visual/arm4.dae"/>
+                    <mesh filename="package://kuka_youbot_support/meshes/visual/link_4.dae"/>
                 </geometry>
             </visual>
@@ -382,12 +297,12 @@
                 <origin xyz="0 -0.010 0.029" rpy="0 0 0"/>
                 <geometry>
-                    <mesh filename="package://kuka_youbot_support/meshes/collision/arm4_convex.dae"/>
-                </geometry>
-            </collision>
-        </link>
-         <link name="${prefix}arm_link_5">
-            <inertial>
-                <mass value="${link_5_mass}"/>
-                <origin xyz="${0/1000} ${1.15/1000} ${-16.83/1000}"
+                    <mesh filename="package://kuka_youbot_support/meshes/collision/link_4.stl"/>
+                </geometry>
+            </collision>
+        </link>
+        <link name="${prefix}arm_link_5">
+            <inertial>
+                <mass value="0.251"/>
+                <origin xyz="0 0.00115 -0.01683"
                         rpy="0 0 0"/>
                 <inertia ixx="0.000280" ixy="0.000000" ixz="0.000000" iyy="0.000339" iyz="0.000000" izz="0.000119"/>
@@ -396,5 +311,5 @@
                 <origin xyz="0.003 0 -0.034" rpy="0 0 0"/>
                 <geometry>
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
File: kuka_youbot_support/urdf/kuka_youbot_transmission.xacro (robot description, xacro)
@@ -1,3 +1,3 @@
-<?xml version="1.0"?>
+<?xml version="1.0"  encoding="UTF-8" ?>
 <robot xmlns:xacro="http://wiki.ros.org/xacro">
     <xacro:macro name="kuka_youbot_transmission" params="prefix control_type">
