Commit message: v0.3

File: kuka_iiwa_14_support/urdf/kuka_iiwa_14_transmission.xacro (robot description, xacro)
@@ -7,8 +7,5 @@
                 <hardwareInterface>hardware_interface/${control_type}JointInterface</hardwareInterface>
             </joint>
-            <actuator name="${prefix}motor1">
-                <hardwareInterface>hardware_interface/${control_type}JointInterface</hardwareInterface>
-                <mechanicalReduction>1</mechanicalReduction>
-            </actuator>
+            <actuator name="${prefix}motor1"/>
         </transmission>
         <transmission name="${prefix}tran2">
@@ -17,8 +14,5 @@
                 <hardwareInterface>hardware_interface/${control_type}JointInterface</hardwareInterface>
             </joint>
-            <actuator name="${prefix}motor2">
-                <hardwareInterface>hardware_interface/${control_type}JointInterface</hardwareInterface>
-                <mechanicalReduction>1</mechanicalReduction>
-            </actuator>
+            <actuator name="${prefix}motor2"/>
         </transmission>
         <transmission name="${prefix}tran3">
@@ -27,8 +21,5 @@
                 <hardwareInterface>hardware_interface/${control_type}JointInterface</hardwareInterface>
             </joint>
-            <actuator name="${prefix}motor3">
-                <hardwareInterface>hardware_interface/${control_type}JointInterface</hardwareInterface>
-                <mechanicalReduction>1</mechanicalReduction>
-            </actuator>
+            <actuator name="${prefix}motor3"/>
         </transmission>
         <transmission name="${prefix}tran4">
@@ -37,8 +28,5 @@
                 <hardwareInterface>hardware_interface/${control_type}JointInterface</hardwareInterface>
             </joint>
-            <actuator name="${prefix}motor4">
-                <hardwareInterface>hardware_interface/${control_type}JointInterface</hardwareInterface>
-                <mechanicalReduction>1</mechanicalReduction>
-            </actuator>
+            <actuator name="${prefix}motor4"/>
         </transmission>
         <transmission name="${prefix}tran5">
@@ -47,8 +35,5 @@
                 <hardwareInterface>hardware_interface/${control_type}JointInterface</hardwareInterface>
             </joint>
-            <actuator name="${prefix}motor5">
-                <hardwareInterface>hardware_interface/${control_type}JointInterface</hardwareInterface>
-                <mechanicalReduction>1</mechanicalReduction>
-            </actuator>
+            <actuator name="${prefix}motor5"/>
         </transmission>
         <transmission name="${prefix}tran6">
@@ -57,8 +42,5 @@
                 <hardwareInterface>hardware_interface/${control_type}JointInterface</hardwareInterface>
             </joint>
-            <actuator name="${prefix}motor6">
-                <hardwareInterface>hardware_interface/${control_type}JointInterface</hardwareInterface>
-                <mechanicalReduction>1</mechanicalReduction>
-            </actuator>
+            <actuator name="${prefix}motor6"/>
         </transmission>
         <transmission name="${prefix}tran7">
@@ -67,8 +49,5 @@
                 <hardwareInterface>hardware_interface/${control_type}JointInterface</hardwareInterface>
             </joint>
-            <actuator name="${prefix}motor7">
-                <hardwareInterface>hardware_interface/${control_type}JointInterface</hardwareInterface>
-                <mechanicalReduction>1</mechanicalReduction>
-            </actuator>
+            <actuator name="${prefix}motor7"/>
         </transmission>
     </xacro:macro>

File: kuka_youbot_support/urdf/kuka_youbot_macro.xacro (robot description, xacro)
@@ -331,5 +331,5 @@
             <child link="${prefix}arm_link_1"/>
             <axis xyz="0 0 -1"/>
-            <dynamics damping="1" friction="1"/>
+            <dynamics damping="0.05" friction="0.05"/>
             <limit effort="${9.5}" velocity="${PI / 2.0}" lower="0" upper="${PI * (169 + 169) / 180}"/>
         </joint>
@@ -339,5 +339,5 @@
             <child link="${prefix}arm_link_2"/>
             <axis xyz="0 1 0"/>
-            <dynamics damping="1" friction="1"/>
+            <dynamics damping="0.05" friction="0.05"/>
             <limit effort="${9.5}" velocity="${PI / 2.0}" lower="0" upper="${PI * (90 + 65) / 180}"/>
         </joint>
@@ -347,5 +347,5 @@
             <child link="${prefix}arm_link_3"/>
             <axis xyz="0 1 0"/>
-            <dynamics damping="1" friction="1"/>
+            <dynamics damping="0.05" friction="0.05"/>
             <limit effort="${6}" velocity="${PI / 2.0}" lower="-${PI * (146 + 151) / 180}" upper="0"/>
         </joint>
@@ -355,5 +355,5 @@
             <child link="${prefix}arm_link_4"/>
             <axis xyz="0 1 0"/>
-            <dynamics damping="1" friction="1"/>
+            <dynamics damping="0.05" friction="0.05"/>
             <limit effort="${2}" velocity="${PI / 2.0}" lower="0" upper="${PI * (102.5 + 102.5) / 180}"/>
         </joint>
@@ -363,5 +363,5 @@
             <child link="${prefix}arm_link_5"/>
             <axis xyz="0 0 -1"/>
-            <dynamics damping="1" friction="1"/>
+            <dynamics damping="0.05" friction="0.05"/>
             <limit effort="1" velocity="${PI / 2.0}" lower="0" upper="${PI * (167.5 + 167.5) / 180}"/>
         </joint>

File: kuka_youbot_support/urdf/kuka_youbot_transmission.xacro (robot description, xacro)
@@ -5,8 +5,5 @@
         <transmission name="${prefix}arm_trans_1">
             <type>transmission_interface/SimpleTransmission</type>
-            <actuator name="${prefix}arm_motor_1">
-                <hardwareInterface>hardware_interface/${control_type}JointInterface</hardwareInterface>
-                <mechanicalReduction>1</mechanicalReduction>
-            </actuator>
+            <actuator name="${prefix}arm_motor_1"/>
             <joint name="${prefix}arm_joint_1">
                 <hardwareInterface>hardware_interface/${control_type}JointInterface</hardwareInterface>
@@ -15,8 +12,5 @@
         <transmission name="${prefix}arm_trans_2">
             <type>transmission_interface/SimpleTransmission</type>
-            <actuator name="${prefix}arm_motor_2">
-                <hardwareInterface>hardware_interface/${control_type}JointInterface</hardwareInterface>
-                <mechanicalReduction>1</mechanicalReduction>
-            </actuator>
+            <actuator name="${prefix}arm_motor_2"/>
             <joint name="${prefix}arm_joint_2">
                 <hardwareInterface>hardware_interface/${control_type}JointInterface</hardwareInterface>
@@ -25,8 +19,5 @@
         <transmission name="${prefix}arm_trans_3">
             <type>transmission_interface/SimpleTransmission</type>
-            <actuator name="${prefix}arm_motor_3">
-                <hardwareInterface>hardware_interface/${control_type}JointInterface</hardwareInterface>
-                <mechanicalReduction>1</mechanicalReduction>
-            </actuator>
+            <actuator name="${prefix}arm_motor_3"/>
             <joint name="${prefix}arm_joint_3">
                 <hardwareInterface>hardware_interface/${control_type}JointInterface</hardwareInterface>
@@ -35,8 +26,5 @@
         <transmission name="${prefix}arm_trans_4">
             <type>transmission_interface/SimpleTransmission</type>
-            <actuator name="${prefix}arm_motor_4">
-                <hardwareInterface>hardware_interface/${control_type}JointInterface</hardwareInterface>
-                <mechanicalReduction>1</mechanicalReduction>
-            </actuator>
+            <actuator name="${prefix}arm_motor_4"/>
             <joint name="${prefix}arm_joint_4">
                 <hardwareInterface>hardware_interface/${control_type}JointInterface</hardwareInterface>
@@ -45,8 +33,5 @@
         <transmission name="${prefix}arm_trans_5">
             <type>transmission_interface/SimpleTransmission</type>
-            <actuator name="${prefix}arm_motor_5">
-                <hardwareInterface>hardware_interface/${control_type}JointInterface</hardwareInterface>
-                <mechanicalReduction>1</mechanicalReduction>
-            </actuator>
+            <actuator name="${prefix}arm_motor_5"/>
             <joint name="${prefix}arm_joint_5">
                 <hardwareInterface>hardware_interface/${control_type}JointInterface</hardwareInterface>
@@ -58,8 +43,5 @@
         <transmission name="${prefix}wheel_trans_fl">
             <type>transmission_interface/SimpleTransmission</type>
-            <actuator name="${prefix}wheel_motor_fl">
-                <hardwareInterface>hardware_interface/VelocityJointInterface</hardwareInterface>
-                <mechanicalReduction>${wheel_mechanical_reduction}</mechanicalReduction>
-            </actuator>
+            <actuator name="${prefix}wheel_motor_fl"/>
             <joint name="${prefix}wheel_joint_fl">
                 <hardwareInterface>hardware_interface/VelocityJointInterface</hardwareInterface>
@@ -68,8 +50,5 @@
         <transmission name="${prefix}caster_trans_fl">
             <type>transmission_interface/SimpleTransmission</type>
-            <actuator name="${prefix}caster_motor_fl">
-                <hardwareInterface>hardware_interface/VelocityJointInterface</hardwareInterface>
-                <mechanicalReduction>${caster_mechanical_reduction}</mechanicalReduction>
-            </actuator>
+            <actuator name="${prefix}caster_motor_fl"/>
             <joint name="${prefix}caster_joint_fl">
                 <hardwareInterface>hardware_interface/VelocityJointInterface</hardwareInterface>
@@ -78,8 +57,5 @@
         <transmission name="${prefix}wheel_trans_fr">
             <type>transmission_interface/SimpleTransmission</type>
-            <actuator name="${prefix}wheel_motor_fr">
-                <hardwareInterface>hardware_interface/VelocityJointInterface</hardwareInterface>
-                <mechanicalReduction>${wheel_mechanical_reduction}</mechanicalReduction>
-            </actuator>
+            <actuator name="${prefix}wheel_motor_fr"/>
             <joint name="${prefix}wheel_joint_fr">
                 <hardwareInterface>hardware_interface/VelocityJointInterface</hardwareInterface>
@@ -88,8 +64,5 @@
         <transmission name="${prefix}caster_trans_fr">
             <type>transmission_interface/SimpleTransmission</type>
-            <actuator name="${prefix}caster_motor_fr">
-                <hardwareInterface>hardware_interface/VelocityJointInterface</hardwareInterface>
-                <mechanicalReduction>${caster_mechanical_reduction}</mechanicalReduction>
-            </actuator>
+            <actuator name="${prefix}caster_motor_fr"/>
             <joint name="${prefix}caster_joint_fr">
                 <hardwareInterface>hardware_interface/VelocityJointInterface</hardwareInterface>
@@ -98,8 +71,5 @@
         <transmission name="${prefix}wheel_trans_bl">
             <type>transmission_interface/SimpleTransmission</type>
-            <actuator name="${prefix}wheel_motor_bl">
-                <hardwareInterface>hardware_interface/VelocityJointInterface</hardwareInterface>
-                <mechanicalReduction>${wheel_mechanical_reduction}</mechanicalReduction>
-            </actuator>
+            <actuator name="${prefix}wheel_motor_bl"/>
             <joint name="${prefix}wheel_joint_bl">
                 <hardwareInterface>hardware_interface/VelocityJointInterface</hardwareInterface>
@@ -108,8 +78,5 @@
         <transmission name="${prefix}caster_trans_bl">
             <type>transmission_interface/SimpleTransmission</type>
-            <actuator name="${prefix}caster_motor_bl">
-                <hardwareInterface>hardware_interface/VelocityJointInterface</hardwareInterface>
-                <mechanicalReduction>${caster_mechanical_reduction}</mechanicalReduction>
-            </actuator>
+            <actuator name="${prefix}caster_motor_bl"/>
             <joint name="${prefix}caster_joint_bl">
                 <hardwareInterface>hardware_interface/VelocityJointInterface</hardwareInterface>
@@ -118,8 +85,5 @@
         <transmission name="${prefix}wheel_trans_br">
             <type>transmission_interface/SimpleTransmission</type>
-            <actuator name="${prefix}wheel_motor_br">
-                <hardwareInterface>hardware_interface/VelocityJointInterface</hardwareInterface>
-                <mechanicalReduction>${wheel_mechanical_reduction}</mechanicalReduction>
-            </actuator>
+            <actuator name="${prefix}wheel_motor_br"/>
             <joint name="${prefix}wheel_joint_br">
                 <hardwareInterface>hardware_interface/VelocityJointInterface</hardwareInterface>
@@ -128,8 +92,5 @@
         <transmission name="${prefix}caster_trans_br">
             <type>transmission_interface/SimpleTransmission</type>
-            <actuator name="${prefix}caster_motor_br">
-                <hardwareInterface>hardware_interface/VelocityJointInterface</hardwareInterface>
-                <mechanicalReduction>${caster_mechanical_reduction}</mechanicalReduction>
-            </actuator>
+            <actuator name="${prefix}caster_motor_br"/>
             <joint name="${prefix}caster_joint_br">
                 <hardwareInterface>hardware_interface/VelocityJointInterface</hardwareInterface>
@@ -139,8 +100,5 @@
         <transmission name="${prefix}gripper_finger_l_trans">
             <type>transmission_interface/SimpleTransmission</type>
-            <actuator name="${prefix}gripper_finger_l_motor">
-                <hardwareInterface>EffortJointInterface</hardwareInterface>
-                <mechanicalReduction>hardware_interface/${control_type}JointInterface</mechanicalReduction>
-            </actuator>
+            <actuator name="${prefix}gripper_finger_l_motor"/>
             <joint name="${prefix}gripper_finger_joint_l">
                 <hardwareInterface>hardware_interface/${control_type}JointInterface</hardwareInterface>
@@ -149,8 +107,5 @@
         <transmission name="${prefix}gripper_finger_r_trans">
             <type>transmission_interface/SimpleTransmission</type>
-            <actuator name="${prefix}gripper_finger_r_motor">
-                <hardwareInterface>hardware_interface/${control_type}JointInterface</hardwareInterface>
-                <mechanicalReduction>1</mechanicalReduction>
-            </actuator>
+            <actuator name="${prefix}gripper_finger_r_motor"/>
             <joint name="${prefix}gripper_finger_joint_r">
                 <hardwareInterface>hardware_interface/${control_type}JointInterface</hardwareInterface>
