Commit message: v0.4

File: kuka_youbot_support/urdf/kuka_youbot_macro.xacro (robot description, xacro)
@@ -430,19 +430,13 @@
             <child link="${prefix}_palm_link"/>
         </joint>
-        <joint name="${prefix}gripper_finger_joint_l" type="prismatic">
+        <joint name="${prefix}gripper_finger_joint_l" type="fixed">
             <origin xyz="0.004 0.008 0.046" rpy="0 0 ${PI}"/>
             <parent link="${prefix}_palm_link"/>
             <child link="${prefix}gripper_finger_link_l"/>
-            <axis xyz="0 -1 0"/>
-            <dynamics damping="1.0" friction="1.0"/>
-            <limit effort="1" velocity="0.1" lower="0" upper="0.0115"/>
-        </joint>
-        <joint name="${prefix}gripper_finger_joint_r" type="prismatic">
+        </joint>
+        <joint name="${prefix}gripper_finger_joint_r" type="fixed">
             <origin xyz="0.004 -0.008 0.046" rpy="0 0 0"/>
             <parent link="${prefix}_palm_link"/>
             <child link="${prefix}gripper_finger_link_r"/>
-            <axis xyz="0 -1 0"/>
-            <dynamics damping="1.0" friction="1.0"/>
-            <limit effort="1" velocity="0.1" lower="0" upper="0.0115"/>
         </joint>
     </xacro:macro>

File: kuka_youbot_support/urdf/kuka_youbot_transmission.xacro (robot description, xacro)
@@ -97,19 +97,4 @@
             </joint>
         </transmission>
-        <!--**************************GRIPPER************************************-->
-        <transmission name="${prefix}gripper_finger_l_trans">
-            <type>transmission_interface/SimpleTransmission</type>
-            <actuator name="${prefix}gripper_finger_l_motor"/>
-            <joint name="${prefix}gripper_finger_joint_l">
-                <hardwareInterface>hardware_interface/${control_type}JointInterface</hardwareInterface>
-            </joint>
-        </transmission>
-        <transmission name="${prefix}gripper_finger_r_trans">
-            <type>transmission_interface/SimpleTransmission</type>
-            <actuator name="${prefix}gripper_finger_r_motor"/>
-            <joint name="${prefix}gripper_finger_joint_r">
-                <hardwareInterface>hardware_interface/${control_type}JointInterface</hardwareInterface>
-            </joint>
-        </transmission>
     </xacro:macro>
 </robot>
